File: Alish40V1.2/40% Alice.kicad_pcb (KiCad board)
At the start: 2 copper layers, 329.7 x 104.5 mm, 96 parts, among them J1 Conn_01x03, K1 KEYSW, K10 KEYSW, K11 KEYSW, K12 KEYSW, K13 KEYSW, K14 KEYSW, K15 KEYSW, K16 KEYSW, K17 KEYSW, K18 KEYSW, K19 KEYSW, K2 KEYSW, K20 KEYSW, K21 KEYSW, K22 KEYSW, K23 KEYSW, K24 KEYSW, K25 KEYSW, K26 KEYSW, K27 KEYSW, K28 KEYSW, K29 KEYSW, K3 KEYSW, K30 KEYSW, K31 KEYSW, K32 KEYSW, K33 KEYSW, K34 KEYSW, K35 KEYSW, K36 KEYSW, K37 KEYSW, K38 KEYSW, K39 KEYSW, K4 KEYSW, K40 KEYSW, K41 KEYSW, K42 KEYSW, K43 KEYSW, K44 KEYSW, K45 KEYSW, K46 KEYSW, K47 KEYSW, K5 KEYSW, K6 KEYSW, K7 KEYSW, K8 KEYSW, K9 KEYSW, U1 ProMicro

Commit message: Updated all files
New artwork, fixed traces and footprints on wrong side of board, included backplate
Parts:
- D37: moved to B.Cu
Routing:
- net ROW5: track 284.9 -> 274.6 mm
- net ROW7: track 317.4 -> 314.8 mm
- net ROW6: track 279.6 -> 281.3 mm
- net COL6: track 305.5 -> 304.3 mm
- net VCC: track 111.4 -> 110.8 mm
- net ENCODER 2: track 118.1 -> 117.5 mm

Commit message: Updated PCB and Schematic
Changed Reference Designators, updated footprints, fixed several routing issues, added Reed X (silly), added my footprints, moved encoder slightly, tightened up QAZ to WSX spacing.
Parts:
- removed the G*** at (217.2, 156.5)
- added G***: LOGO, LOGO, F.Cu at (218.1, 155.8)
- added G***: LOGO, LOGO, B.Cu at (108.3, 84.9)
- MX1: renamed from K1; footprint Button_Switch_Keyboard:SW_Cherry_MX_1.50u_PCB -> ReedsKeebs:1.5U MX
- MX10: renamed from K10; footprint Button_Switch_Keyboard:SW_Cherry_MX_1.00u_PCB -> ReedsKeebs:1U MX
- MX11: renamed from K11; footprint Button_Switch_Keyboard:SW_Cherry_MX_1.00u_PCB -> ReedsKeebs:1U MX
- MX12: renamed from K12; footprint Button_Switch_Keyboard:SW_Cherry_MX_1.50u_PCB -> ReedsKeebs:1.5U MX
- MX13: renamed from K13; footprint Button_Switch_Keyboard:SW_Cherry_MX_1.75u_PCB -> ReedsKeebs:1.75U MX
- MX14: renamed from K14; footprint Button_Switch_Keyboard:SW_Cherry_MX_1.00u_PCB -> ReedsKeebs:1U MX
- MX15: renamed from K15; footprint Button_Switch_Keyboard:SW_Cherry_MX_1.00u_PCB -> ReedsKeebs:1U MX
- MX16: renamed from K16; footprint Button_Switch_Keyboard:SW_Cherry_MX_1.00u_PCB -> ReedsKeebs:1U MX
- MX17: renamed from K17; footprint Button_Switch_Keyboard:SW_Cherry_MX_1.00u_PCB -> ReedsKeebs:1U MX
- MX18: renamed from K18; footprint Button_Switch_Keyboard:SW_Cherry_MX_1.00u_PCB -> ReedsKeebs:1U MX
- MX19: renamed from K19; footprint Button_Switch_Keyboard:SW_Cherry_MX_1.00u_PCB -> ReedsKeebs:1U MX
- MX2: renamed from K2; footprint Button_Switch_Keyboard:SW_Cherry_MX_1.00u_PCB -> ReedsKeebs:1U MX
- MX20: renamed from K20; footprint Button_Switch_Keyboard:SW_Cherry_MX_1.00u_PCB -> ReedsKeebs:1U MX
- MX21: renamed from K21; footprint Button_Switch_Keyboard:SW_Cherry_MX_1.00u_PCB -> ReedsKeebs:1U MX
- MX22: renamed from K22; footprint Button_Switch_Keyboard:SW_Cherry_MX_1.00u_PCB -> ReedsKeebs:1U MX
- MX23: renamed from K23; footprint Button_Switch_Keyboard:SW_Cherry_MX_1.00u_PCB -> ReedsKeebs:1U MX
- MX24: renamed from K24; footprint Button_Switch_Keyboard:SW_Cherry_MX_1.25u_PCB -> ReedsKeebs:1.25U MX
- MX24-1: renamed from K25; footprint Button_Switch_Keyboard:SW_Cherry_MX_2.25u_PCB -> ReedsKeebs:2.25U MX
- MX25: renamed from K26; footprint Button_Switch_Keyboard:SW_Cherry_MX_2.25u_PCB -> ReedsKeebs:2.25U MX
- MX25-1: renamed from K38; footprint Button_Switch_Keyboard:SW_Cherry_MX_1.25u_PCB -> ReedsKeebs:1.25U MX
- MX26: renamed from K27; footprint Button_Switch_Keyboard:SW_Cherry_MX_1.00u_PCB -> ReedsKeebs:1U MX
- MX27: renamed from K28; footprint Button_Switch_Keyboard:SW_Cherry_MX_1.00u_PCB -> ReedsKeebs:1U MX
- MX28: renamed from K29; footprint Button_Switch_Keyboard:SW_Cherry_MX_1.00u_PCB -> ReedsKeebs:1U MX
- MX29: renamed from K30; footprint Button_Switch_Keyboard:SW_Cherry_MX_1.00u_PCB -> ReedsKeebs:1U MX
- MX3: renamed from K3; footprint Button_Switch_Keyboard:SW_Cherry_MX_1.00u_PCB -> ReedsKeebs:1U MX
- MX30: renamed from K31; footprint Button_Switch_Keyboard:SW_Cherry_MX_1.00u_PCB -> ReedsKeebs:1U MX
- MX31: renamed from K32; footprint Button_Switch_Keyboard:SW_Cherry_MX_1.00u_PCB -> ReedsKeebs:1U MX
- MX32: renamed from K33; footprint Button_Switch_Keyboard:SW_Cherry_MX_1.00u_PCB -> ReedsKeebs:1U MX
- MX33: renamed from K34; footprint Button_Switch_Keyboard:SW_Cherry_MX_1.00u_PCB -> ReedsKeebs:1U MX
- MX34: renamed from K35; footprint Button_Switch_Keyboard:SW_Cherry_MX_1.00u_PCB -> ReedsKeebs:1U MX
- MX35: renamed from K36; footprint Button_Switch_Keyboard:SW_Cherry_MX_1.00u_PCB -> ReedsKeebs:1U MX
- MX36: renamed from K37; footprint Button_Switch_Keyboard:SW_Cherry_MX_1.75u_PCB -> ReedsKeebs:1.75U MX
- MX37: renamed from K40; footprint Button_Switch_Keyboard:SW_Cherry_MX_1.25u_PCB -> ReedsKeebs:1.25U MX
- MX38: renamed from K41; footprint Button_Switch_Keyboard:SW_Cherry_MX_1.25u_PCB -> ReedsKeebs:1.25U MX
- MX39: renamed from K42; footprint Button_Switch_Keyboard:SW_Cherry_MX_1.25u_PCB -> ReedsKeebs:1.25U MX
- MX4: renamed from K4; footprint Button_Switch_Keyboard:SW_Cherry_MX_1.00u_PCB -> ReedsKeebs:1U MX
- MX40: renamed from K39; footprint Button_Switch_Keyboard:SW_Cherry_MX_1.00u_PCB -> ReedsKeebs:1U MX
- MX41: renamed from K43; footprint Button_Switch_Keyboard:SW_Cherry_MX_2.25u_PCB -> ReedsKeebs:2.25U MX
- MX42: renamed from K44; footprint Button_Switch_Keyboard:SW_Cherry_MX_2.75u_PCB -> ReedsKeebs:SW_Cherry_MX_2.75u_PCB
- MX43: renamed from K45; footprint Button_Switch_Keyboard:SW_Cherry_MX_1.25u_PCB -> ReedsKeebs:1.25U MX
- MX44: renamed from K46; footprint Button_Switch_Keyboard:SW_Cherry_MX_1.25u_PCB -> ReedsKeebs:1.25U MX
- MX45: renamed from K47; footprint Button_Switch_Keyboard:SW_Cherry_MX_1.25u_PCB -> ReedsKeebs:1.25U MX
- MX5: renamed from K5; footprint Button_Switch_Keyboard:SW_Cherry_MX_1.00u_PCB -> ReedsKeebs:1U MX
- MX6: renamed from K6; footprint Button_Switch_Keyboard:SW_Cherry_MX_1.00u_PCB -> ReedsKeebs:1U MX
- MX7: renamed from K7; footprint Button_Switch_Keyboard:SW_Cherry_MX_1.00u_PCB -> ReedsKeebs:1U MX
- MX8: renamed from K8; footprint Button_Switch_Keyboard:SW_Cherry_MX_1.00u_PCB -> ReedsKeebs:1U MX
- MX9: renamed from K9; footprint Button_Switch_Keyboard:SW_Cherry_MX_1.00u_PCB -> ReedsKeebs:1U MX
- moved D2 5.62 mm to (118.2, 91.4)
- moved MX1 3.42 mm to (85.2, 94.8)
- moved MX2 3.38 mm to (109.0, 94.8)
- moved D44 3.14 mm to (321.5, 146.1)
- moved MX12 2.90 mm to (346.7, 92.9)
- moved MX11 2.69 mm to (323.0, 92.9)
- moved MX13 2.05 mm to (84.3, 113.8)
- moved MX14 2.04 mm to (110.5, 113.8)
- moved D11 1.85 mm to (311.8, 91.9)
- moved D23 1.48 mm to (318.6, 110.0)
- moved J1 1.45 mm to (314.9, 118.9)
- moved MX24-1 1.39 mm to (342.9, 112.0)
- moved MX24 1.38 mm to (352.4, 112.0)
- moved MX23 1.35 mm to (331.0, 112.0)
- moved MX44 0.15 mm to (333.1, 150.2)
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- renumbered D38 to D37, D39 to D38, D40 to D39, D37 to D40
Routing:
- net COL1: track 277.3 -> 271.1 mm
- net ROW2: track 277.9 -> 272.2 mm
- net ROW8: track 281.5 -> 285.1 mm
- net Net-(D1-Pad2): track 10.9 -> 7.51 mm
- net Net-(D44-Pad2): track 8.71 -> 5.66 mm
- net Net-(D12-Pad2): track 9.07 -> 6.21 mm
- net Net-(D2-Pad2): track 8.81 -> 11.4 mm
- net ROW1: track 262.3 -> 260.2 mm
- net Net-(D13-Pad2): track 11.6 -> 9.53 mm
- net Net-(D14-Pad2): track 9.32 -> 7.29 mm
- net RGB DIN: track 105.2 -> 103.3 mm
- net Net-(D8-Pad2): track 5.93 -> 4.45 mm
- net ROW3: track 269.9 -> 268.4 mm
- net VCC: track 110.8 -> 109.3 mm
- net ENCODER 1: track 113.5 -> 112.1 mm
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