File: Alish40V1.2/alish40/40% Alice.kicad_pcb (KiCad board)
At the start: 2 copper layers, 329.7 x 104.5 mm, 97 parts, among them J1 Conn_01x03, U1 ProMicro

Commit message: redo everything lmao
Parts:
- J1: moved to B.Cu
- moved D25 20.9 mm to (94.2, 109.9)
- moved D38 19.3 mm to (90.5, 136.1)
- moved D31 16.3 mm to (256.5, 126.2)
- moved D32 16.1 mm to (259.0, 125.7)
- moved D23 15.9 mm to (327.1, 96.7)
- moved D11 15.0 mm to (319.8, 79.3)
- moved D35 14.8 mm to (319.8, 115.6)
- moved D34 14.4 mm to (296.6, 119.0)
- moved D33 14.3 mm to (277.7, 122.3)
- moved D21 14.2 mm to (283.6, 101.9)
- moved D45 14.1 mm to (349.9, 134.7)
- moved D22 14.0 mm to (302.1, 98.6)
- moved D24 13.9 mm to (342.8, 89.1)
- moved D36 13.8 mm to (345.1, 115.2)
- moved D42 13.7 mm to (288.4, 142.9)
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Connections:
- D18 pad 2: Net-(D18-Pad2) -> Net-(MX18-Pad2)
- D19 pad 2: Net-(D19-Pad2) -> Net-(MX19-Pad1)
- D30 pad 2: Net-(D30-Pad2) -> Net-(MX30-Pad2)
- D31 pad 2: Net-(D31-Pad2) -> Net-(MX31-Pad1)
- D38 pad 2: Net-(D38-Pad2) -> Net-(MX38-Pad2)
- D41 pad 2: Net-(D41-Pad2) -> Net-(MX41-Pad2)
- D42 pad 2: Net-(D42-Pad2) -> Net-(MX42-Pad1)
- D6 pad 2: Net-(D6-Pad2) -> Net-(MX6-Pad2)
- D7 pad 2: Net-(D7-Pad2) -> Net-(MX7-Pad1)
- J1 pad 1: VCC -> GND
- J1 pad 3: GND -> VCC
- MX18 pad 1: Net-(D18-Pad2) -> COL3
- MX18 pad 2: COL3 -> Net-(MX18-Pad2)
- MX19 pad 1: COL4 -> Net-(MX19-Pad1)
- MX19 pad 2: Net-(D19-Pad2) -> COL4
- MX30 pad 1: Net-(D30-Pad2) -> COL3
- MX30 pad 2: COL3 -> Net-(MX30-Pad2)
- MX31 pad 1: COL4 -> Net-(MX31-Pad1)
- MX31 pad 2: Net-(D31-Pad2) -> COL4
- MX38 pad 1: Net-(D38-Pad2) -> COL1
- MX38 pad 2: COL1 -> Net-(MX38-Pad2)
- MX41 pad 1: Net-(D41-Pad2) -> COL3
- MX41 pad 2: COL3 -> Net-(MX41-Pad2)
- MX42 pad 1: COL4 -> Net-(MX42-Pad1)
- MX42 pad 2: Net-(D42-Pad2) -> COL4
- MX6 pad 1: Net-(D6-Pad2) -> COL3
- MX6 pad 2: COL3 -> Net-(MX6-Pad2)
- MX7 pad 1: COL4 -> Net-(MX7-Pad1)
- MX7 pad 2: Net-(D7-Pad2) -> COL4
- U1 pad 1: COL1 -> COL2
- U1 pad 10: ROW2 -> ROW5
- U1 pad 11: ROW3 -> ROW7
- U1 pad 12: ROW4 -> ROW8
- U1 pad 13: ROW5 -> COL4
- U1 pad 14: ROW6 -> COL6
- U1 pad 15: ROW7 -> COL5
- U1 pad 16: ROW8 -> COL3
- U1 pad 17: ENCODER 2 -> unconnected-(U1-Pad17)
- U1 pad 18: ENCODER 1 -> ENCODER 2
- U1 pad 19: unconnected-(U1-Pad19) -> ENCODER 1
- U1 pad 2: COL2 -> COL1
- U1 pad 5: COL3 -> ROW1
- U1 pad 6: COL4 -> ROW2
- U1 pad 7: COL5 -> ROW3
- U1 pad 8: COL6 -> ROW4
- U1 pad 9: ROW1 -> ROW6
Routing:
- net ROW1: track 262.0 -> 307.7 mm, vias 0 -> 1
- net COL3: track 151.7 -> 194.3 mm, vias 0 -> 3
- net ROW8: track 288.7 -> 324.1 mm, vias 0 -> 1
- net ROW2: track 273.6 -> 304.6 mm, vias 0 -> 1
- net COL6: track 299.9 -> 272.2 mm, vias 1 -> 2
- net Net-(D42-Pad2): track 24.8 -> 0.00 mm
- net Net-(D41-Pad2): track 24.3 -> 0.00 mm
- net Net-(MX42-Pad1): track 0.00 -> 23.1 mm
- net ROW3: track 260.0 -> 282.2 mm
- net ROW4: track 250.8 -> 272.4 mm, vias 2 -> 1
- net Net-(MX41-Pad2): track 0.00 -> 17.4 mm
- net COL2: track 242.5 -> 258.8 mm
- net RGB DIN: track 109.9 -> 125.9 mm, vias 0 -> 2
- net COL1: track 271.6 -> 287.4 mm
- net Net-(D25-Pad2): track 32.5 -> 17.3 mm
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Other:
- outline, holes or cut-outs redrawn
