File: Alish40V1.2/alish40/40% Alice.kicad_sch (KiCad schematic)
At the start: 95 parts, among them J1 Conn_01x03, U1 ProMicro

Commit message: redo everything lmao
Connections:
- net COL1: now also MX38.1, U1.2 (RX); no longer MX38.2, U1.1 (TX)
- net COL2: now also U1.1 (TX); no longer U1.2 (RX)
- net COL3: now also MX18.1, MX30.1, MX41.1, MX6.1, U1.16 (B1); no longer MX18.2, MX30.2, MX41.2, MX6.2, U1.5 (SDA)
- net COL4: now also MX19.2, MX31.2, MX42.2, MX7.2, U1.13 (B6); no longer MX19.1, MX31.1, MX42.1, MX7.1, U1.6 (SCL)
- net COL5: now also U1.15 (B3); no longer U1.7 (D4)
- net COL6: now also U1.14 (B2); no longer U1.8 (C6)
- net ENCODER 1: now also U1.19 (F5); no longer U1.18 (F6)
- net ENCODER 2: now also U1.18 (F6); no longer U1.17 (F7)
- net GND: now also J1.1 (Pin_1); no longer J1.3 (Pin_3)
- net ROW1: now also U1.5 (SDA); no longer U1.9 (D7)
- net ROW2: now also U1.6 (SCL); no longer U1.10 (E6)
- net ROW3: now also U1.7 (D4); no longer U1.11 (B4)
- net ROW4: now also U1.8 (C6); no longer U1.12 (B5)
- net ROW5: now also U1.10 (E6); no longer U1.13 (B6)
- net ROW6: now also U1.9 (D7); no longer U1.14 (B2)
- net ROW7: now also U1.11 (B4); no longer U1.15 (B3)
- net ROW8: now also U1.12 (B5); no longer U1.16 (B1)
- net VCC: now also J1.3 (Pin_3); no longer J1.1 (Pin_1)
- net at D18.2 (A): now also MX18.2; no longer MX18.1
- net at D19.2 (A): now also MX19.1; no longer MX19.2
- net at D7.2 (A): now also MX7.1; no longer MX7.2
- net at D31.2 (A): now also MX31.1; no longer MX31.2
- net at D38.2 (A): now also MX38.2; no longer MX38.1
- net at D41.2 (A): now also MX41.2; no longer MX41.1
- net at D30.2 (A): now also MX30.2; no longer MX30.1
- net at D42.2 (A): now also MX42.1; no longer MX42.2
- net at D6.2 (A): now also MX6.2; no longer MX6.1
Other:
- moved on the sheet: D18, D19, D30, D31, D38, D41, D42, D6, D7
