File: alish40/alish40_6-06/alish40.kicad_pcb (KiCad board)
At the start: 2 copper layers, 329.7 x 104.5 mm, 98 parts, among them J1 Conn_01x03, SW1 SW_SPST, U1 ProMicro

Commit message: final proto finished
Parts:
- added G***: LOGO, MWMX_art:silly2, B.Cu at (88.9, 72.6)
- D1, D10, D11, D12, D13, D14, D15, D16, D17, D18, D19, D2, D20, D21, D22, D23, D24, D25, D26, D27, D28, D29, D3, D30, D31, D32, D33, D34, D35, D36, D4, D41, D42, D43, D44, D45, D5, D6, D7, D8, D9: footprint Diode_THT:D_DO-35_SOD27_P7.62mm_Horizontal -> alish:clean_diode
- D37: renamed from D40; footprint Diode_THT:D_DO-35_SOD27_P7.62mm_Horizontal -> alish:clean_diode
- D38: renamed from D37; footprint Diode_THT:D_DO-35_SOD27_P7.62mm_Horizontal -> alish:clean_diode
- D39: renamed from D38; footprint Diode_THT:D_DO-35_SOD27_P7.62mm_Horizontal -> alish:clean_diode
- D40: renamed from D39; footprint Diode_THT:D_DO-35_SOD27_P7.62mm_Horizontal -> alish:clean_diode
- MX1, MX10, MX11, MX12, MX13, MX14, MX15, MX16, MX17, MX18, MX19, MX2, MX20, MX21, MX22, MX23, MX24, MX24-1, MX25, MX25-1, MX3, MX4, MX41, MX42, MX43, MX44, MX45, MX5, MX6, MX7, MX8, MX9: footprint Button_Switch_Keyboard:SW_Cherry_MX_1.00u_PCB -> alish:SW_Cherry_MX_1.00u_PCB
- MX26: renamed from MX40; footprint Button_Switch_Keyboard:SW_Cherry_MX_1.00u_PCB -> alish:SW_Cherry_MX_1.00u_PCB
- MX27: renamed from MX26; footprint Button_Switch_Keyboard:SW_Cherry_MX_1.00u_PCB -> alish:SW_Cherry_MX_1.00u_PCB
- MX28: renamed from MX27; footprint Button_Switch_Keyboard:SW_Cherry_MX_1.00u_PCB -> alish:SW_Cherry_MX_1.00u_PCB
- MX29: renamed from MX28; footprint Button_Switch_Keyboard:SW_Cherry_MX_1.00u_PCB -> alish:SW_Cherry_MX_1.00u_PCB
- MX30: renamed from MX29; footprint Button_Switch_Keyboard:SW_Cherry_MX_1.00u_PCB -> alish:SW_Cherry_MX_1.00u_PCB
- MX31: renamed from MX30; footprint Button_Switch_Keyboard:SW_Cherry_MX_1.00u_PCB -> alish:SW_Cherry_MX_1.00u_PCB
- MX32: renamed from MX31; footprint Button_Switch_Keyboard:SW_Cherry_MX_1.00u_PCB -> alish:SW_Cherry_MX_1.00u_PCB
- MX33: renamed from MX32; footprint Button_Switch_Keyboard:SW_Cherry_MX_1.00u_PCB -> alish:SW_Cherry_MX_1.00u_PCB
- MX34: renamed from MX33; footprint Button_Switch_Keyboard:SW_Cherry_MX_1.00u_PCB -> alish:SW_Cherry_MX_1.00u_PCB
- MX35: renamed from MX34; footprint Button_Switch_Keyboard:SW_Cherry_MX_1.00u_PCB -> alish:SW_Cherry_MX_1.00u_PCB
- MX36: renamed from MX35; footprint Button_Switch_Keyboard:SW_Cherry_MX_1.00u_PCB -> alish:SW_Cherry_MX_1.00u_PCB
- MX37: renamed from MX36; footprint Button_Switch_Keyboard:SW_Cherry_MX_1.00u_PCB -> alish:SW_Cherry_MX_1.00u_PCB
- MX38: renamed from MX37; footprint Button_Switch_Keyboard:SW_Cherry_MX_1.00u_PCB -> alish:SW_Cherry_MX_1.00u_PCB
- MX39: renamed from MX38; footprint Button_Switch_Keyboard:SW_Cherry_MX_1.00u_PCB -> alish:SW_Cherry_MX_1.00u_PCB
- MX40: renamed from MX39; footprint Button_Switch_Keyboard:SW_Cherry_MX_1.00u_PCB -> alish:SW_Cherry_MX_1.00u_PCB
Other:
- outline, holes or cut-outs redrawn
- board text added: "5V-DIN-GND"
- board text added: "JLCJLCJLCJLC"
- board text added: "V1.3"
- board text removed: "V1.2"
