File: alish40/alish40_v1.4/alish40.kicad_pcb (KiCad board)
At the start: 2 copper layers, 329.7 x 104.5 mm, 99 parts, among them J1 Conn_01x03, SW1 SW_SPST, U1 ProMicro

Commit message: modified traces to not be under drill holes
Routing:
- net COL1: track 315.9 -> 321.2 mm
- net Net-(D42-Pad2): track 30.0 -> 34.3 mm
- net ROW8: track 635.5 -> 638.1 mm
- net ROW7: track 608.2 -> 610.7 mm
- net COL3: track 193.8 -> 192.7 mm
